File: ArduinoRobko01/Robko01.kicad_pcb (KiCad board)
At the start: 2 copper layers, 71.1 x 25.4 mm, 12 parts, among them J1 CONN_01X15, J2 CONN_01X15, J3 A, J4 B, J5 C, J6 I2C, J7 UART, J8 SS, J9 SPI

Commit message: Update README
Other:
- board text added: "Orlin Dimitrov, robko01@8bitclub.com"
- board text removed: "Orlin Dimitrov, orlin369@gmail.com"
Changed lines of the file:
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@@
-(kicad_pcb (version 20171130) (host pcbnew "(5.0.2)-1")
+(kicad_pcb (version 20171130) (host pcbnew "(5.1.5)-3")
   (general
     (thickness 1.6)
@@
   )
   (page A4)
+  (title_block
+    (title "Robko01 Arduino Extention")
+    (rev 1.0)
+    (company 8BitClub)
+    (comment 1 "Orlin Dimitrov")
+    (comment 2 robko01@8bitclub.com)
+  )
   (layers
-    (0 F.Cu signal)
-    (31 B.Cu signal)
+    (0 F.Cu signal hide)
+    (31 B.Cu signal hide)
     (32 B.Adhes user)
     (33 F.Adhes user)
@@
     (zone_45_only no)
     (trace_min 0.2)
-    (segment_width 0.2)
-    (edge_width 0.15)
     (via_size 0.6)
     (via_drill 0.4)
@@
     (uvia_min_size 0.2)
     (uvia_min_drill 0.1)
+    (edge_width 0.15)
+    (segment_width 0.2)
     (pcb_text_width 0.3)
     (pcb_text_size 1.5 1.5)
@@
     )
   )
-  (gr_text "Orlin Dimitrov, orlin369@gmail.com" (at 177.8 106.68) (layer B.SilkS)
+  (gr_text "Orlin Dimitrov, robko01@8bitclub.com" (at 177.8 106.68) (layer B.SilkS)
     (effects (font (size 0.8 0.8) (thickness 0.125)) (justify mirror))
   )
-  (gr_text "Orlin Dimitrov, orlin369@gmail.com" (at 177.8 106.68) (layer F.SilkS)
+  (gr_text "Orlin Dimitrov, robko01@8bitclub.com" (at 177.8 106.68) (layer F.SilkS)
     (effects (font (size 0.8 0.8) (thickness 0.125)))
   )

Commit message: Fix main VRM mount holes, connectors naming and labels
Parts:
- moved R2 10.2 mm to (135.6, 124.5), turned to 90 degrees
- moved D1 2.54 mm to (135.6, 109.2), turned to 270 degrees
Connections:
- D1 pad 1: Net-(D1-Pad1) -> LED
- D1 pad 2: LED -> Net-(D1-Pad2)
- R2 pad 1: Net-(D1-Pad1) -> +5V
- R2 pad 2: GND -> Net-(D1-Pad2)
Routing:
- net +5V: track 29.0 -> 43.8 mm
- net Net-(D1-Pad2): track 0.00 -> 2.54 mm
- net Net-(D1-Pad1): track 2.54 -> 0.00 mm
