File: ArduinoRobko01/Robko01.sch (KiCad schematic (older format))
At the start: 12 parts, among them J1 CONN_01X15, J2 CONN_01X15, J3 A, J4 B, J5 C, J6 I2C, J7 UART, J8 SS, J9 SPI

Commit message: Fix main VRM mount holes, connectors naming and labels
Connections:
- net +5V: now also R2.1
- net GND: no longer R2.2
- net LED: now also D1.1 (K); no longer D1.2 (A)
- new net: D1.2 (A), R2.2
Other:
- moved on the sheet: D1, R2
Changed lines of the file:
@@
 EESchema Schematic File Version 4
-LIBS:Robko01-cache
-EELAYER 26 0
+EELAYER 30 0
 EELAYER END
 $Descr A4 11693 8268
@@
 L Device:R R2
 U 1 1 5C0D2DCC
+P 9400 4500
+F 0 "R2" V 9480 4500 50  0000 C CNN
+F 1 "330" V 9300 4500 50  0000 C CNN
+F 2 "Resistors_THT:R_Axial_DIN0207_L6.3mm_D2.5mm_P10.16mm_Horizontal" V 9330 4500 50  0001 C CNN
+F 3 "" H 9400 4500 50  0001 C CNN
+	1    9400 4500
+	1    0    0    -1
+$EndComp
+$Comp
+L Device:LED D1
+U 1 1 5C0D2E40
 P 9400 4900
-F 0 "R2" V 9480 4900 50  0000 C CNN
-F 1 "330" V 9400 4900 50  0000 C CNN
-F 2 "Resistors_THT:R_Axial_DIN0207_L6.3mm_D2.5mm_P10.16mm_Horizontal" V 9330 4900 50  0001 C CNN
+F 0 "D1" H 9400 5000 50  0000 C CNN
+F 1 "LED" H 9400 4800 50  0000 C CNN
+F 2 "LEDs:LED_D3.0mm" H 9400 4900 50  0001 C CNN
 F 3 "" H 9400 4900 50  0001 C CNN
 	1    9400 4900
-	1    0    0    -1
-$EndComp
-$Comp
-L Device:LED D1
-U 1 1 5C0D2E40
-P 9400 4500
-F 0 "D1" H 9400 4600 50  0000 C CNN
-F 1 "LED" H 9400 4400 50  0000 C CNN
-F 2 "LEDs:LED_D3.0mm" H 9400 4500 50  0001 C CNN
-F 3 "" H 9400 4500 50  0001 C CNN
-	1    9400 4500
 	0    -1   -1   0
-$EndComp
-$Comp
-L power:GND #PWR015
-U 1 1 5C0D33C4
-P 9400 5150
-F 0 "#PWR015" H 9400 4900 50  0001 C CNN
-F 1 "GND" H 9400 5000 50  0000 C CNN
-F 2 "" H 9400 5150 50  0001 C CNN
-F 3 "" H 9400 5150 50  0001 C CNN
-	1    9400 5150
-	1    0    0    -1
 $EndComp
 Text GLabel 7850 4100 0    60   Input ~ 0
 LED
-Text GLabel 9300 4250 0    60   Input ~ 0
+Text GLabel 9250 5250 0    60   Input ~ 0
 LED
 NoConn ~ 6350 4200
@@
 	9400 4750 9400 4650
 Wire Wire Line
-	9400 5150 9400 5050
-Wire Wire Line
 	8300 4100 7850 4100
 Wire Wire Line
-	9300 4250 9400 4250
-Wire Wire Line
 	8150 4300 8300 4300
 Wire Wire Line
@@
 Wire Wire Line
 	6100 3250 6100 3500
+Wire Wire Line
+	9250 5250 9400 5250
+Wire Wire Line
+	9400 5250 9400 5050
+$Comp
+L power:+5V #PWR?
+U 1 1 6194C6F7
+P 9400 4250
+F 0 "#PWR?" H 9400 4100 50  0001 C CNN
+F 1 "+5V" H 9400 4390 50  0000 C CNN
+F 2 "" H 9400 4250 50  0001 C CNN
+F 3 "" H 9400 4250 50  0001 C CNN
+	1    9400 4250
+	1    0    0    -1
+$EndComp
 $EndSCHEMATC
